Commit message: unfinished torso repr

File: src/ur5_dual_robot_description/urdf/dual_ur5.urdf.xacro (robot description, xacro)
@@ -1,32 +1,78 @@
 <?xml version="1.0"?>
 <robot xmlns:xacro="http://www.ros.org/wiki/xacro" name="dual_ur5">
-  <!-- Include official UR macro from ur_description package -->
   <xacro:include filename="$(find ur_description)/urdf/ur_macro.xacro"/>
-  <!-- ==================== WORLD & BASE ==================== -->
   <link name="world"/>
-  <!-- Mounting table between the two arms -->
-  <link name="base_platform">
+  <!-- ==================== TORSO STAND ==================== -->
+  <link name="torso_stand">
     <visual>
-      <geometry><box size="1.0 0.5 0.05"/></geometry>
-      <material name="grey"><color rgba="0.5 0.5 0.5 1"/></material>
+      <origin xyz="0 0 0.275"/>
+      <geometry><box size="0.25 0.25 0.55"/></geometry>
+      <material name="dark_grey"><color rgba="0.25 0.25 0.25 1"/></material>
     </visual>
     <collision>
-      <geometry><box size="1.0 0.5 0.05"/></geometry>
+      <origin xyz="0 0 0.275"/>
+      <geometry><box size="0.25 0.25 0.55"/></geometry>
     </collision>
     <inertial>
-      <mass value="20.0"/>
-      <inertia ixx="0.1" ixy="0" ixz="0" iyy="0.1" iyz="0" izz="0.1"/>
+      <mass value="30.0"/>
+      <inertia ixx="0.6" ixy="0" ixz="0" iyy="0.6" iyz="0" izz="0.1"/>
     </inertial>
   </link>
-  <joint name="world_to_platform" type="fixed">
+  <joint name="world_to_stand" type="fixed">
     <parent link="world"/>
-    <child link="base_platform"/>
-    <origin xyz="0 0 -0.025" rpy="0 0 0"/>
+    <child link="torso_stand"/>
+    <origin xyz="0 0 0" rpy="0 0 0"/>
   </joint>
-  <!-- ==================== LEFT ARM (UR5) ==================== -->
-    <xacro:ur_robot
+  <!-- ==================== TORSO BODY ==================== -->
+  <!--
+    Arm attachment points: (±0.22, 0, 1.00) world = (±0.22, 0, 0.45) in torso frame.
+    V-shape mount (viewed from behind, i.e. looking along +Y):
+      Left  arm rpy="${pi} ${-pi/4} 0"  → base Z = [+1/√2, 0, -1/√2]  hangs right+down  (\)
+      Right arm rpy="${pi} ${pi/4}  0"  → base Z = [-1/√2, 0, -1/√2]  hangs left+down   (/)
+    The two arms cross inward forming a V.
+  -->
+  <link name="torso">
+    <visual>
+      <origin xyz="0 0 0.275"/>
+      <geometry><box size="0.44 0.22 0.55"/></geometry>
+      <material name="light_grey"><color rgba="0.75 0.75 0.75 1"/></material>
+    </visual>
+    <collision>
+      <origin xyz="0 0 0.275"/>
+      <geometry><box size="0.44 0.22 0.55"/></geometry>
+    </collision>
+    <inertial>
+      <mass value="15.0"/>
+      <inertia ixx="0.4" ixy="0" ixz="0" iyy="0.4" iyz="0" izz="0.15"/>
+    </inertial>
+  </link>
+  <joint name="stand_to_torso" type="fixed">
+    <parent link="torso_stand"/>
+    <child link="torso"/>
+    <origin xyz="0 0 0.55" rpy="0 0 0"/>
+  </joint>
+  <!-- ==================== HEAD ==================== -->
+  <link name="head">
+    <visual>
+      <origin xyz="0 0 0.11"/>
+      <geometry><sphere radius="0.11"/></geometry>
+      <material name="light_grey"><color rgba="0.75 0.75 0.75 1"/></material>
+    </visual>
+    <inertial>
+      <mass value="2.0"/>
+      <inertia ixx="0.01" ixy="0" ixz="0" iyy="0.01" iyz="0" izz="0.01"/>
+    </inertial>
+  </link>
+  <joint name="torso_to_head" type="fixed">
+    <parent link="torso"/>
+    <child link="head"/>
+    <origin xyz="0 0 0.55" rpy="0 0 0"/>
+  </joint>
+  <!-- ==================== LEFT ARM ==================== -->
+  <!-- Mounted left shoulder, base plate tilted 45° inward (V-shape) -->
+  <xacro:ur_robot
     name="left"
     tf_prefix="left_"
-    parent="world"
+    parent="torso"
     joint_limits_parameters_file="$(find ur_description)/config/ur5/joint_limits.yaml"
     kinematics_parameters_file="$(find ur_description)/config/ur5/default_kinematics.yaml"
@@ -34,10 +80,12 @@
     visual_parameters_file="$(find ur_description)/config/ur5/visual_parameters.yaml"
     generate_ros2_control_tag="false">
-    <origin xyz="-0.35 0 0" rpy="0 0 1.5708"/>
+    <origin xyz="-0.22 0 0.45" rpy="${pi} ${-pi/4} 0"/>
   </xacro:ur_robot>
+  <!-- ==================== RIGHT ARM ==================== -->
+  <!-- Mounted right shoulder, base plate tilted 45° inward (V-shape mirror) -->
   <xacro:ur_robot
     name="right"
     tf_prefix="right_"
-    parent="world"
+    parent="torso"
     joint_limits_parameters_file="$(find ur_description)/config/ur5/joint_limits.yaml"
     kinematics_parameters_file="$(find ur_description)/config/ur5/default_kinematics.yaml"
@@ -45,5 +93,5 @@
     visual_parameters_file="$(find ur_description)/config/ur5/visual_parameters.yaml"
     generate_ros2_control_tag="false">
-    <origin xyz="0.35 0 0" rpy="0 0 ${pi + 1.5708}"/>
+    <origin xyz="0.22 0 0.45" rpy="${pi} ${pi/4} 0"/>
   </xacro:ur_robot>
   <!-- ==================== GRIPPER MACRO ==================== -->
@@ -115,5 +163,4 @@
       <dynamics damping="0.1" friction="0.1"/>
     </joint>
-    <!-- TCP (Tool Center Point) — planning target for IK -->
     <link name="${prefix}tcp"/>
     <joint name="${prefix}tcp_joint" type="fixed">
@@ -123,6 +170,5 @@
     </joint>
   </xacro:macro>
-  <!-- ==================== ATTACH GRIPPERS ==================== -->
-  <xacro:simple_gripper prefix="left_" parent="left_tool0"/>
+  <xacro:simple_gripper prefix="left_"  parent="left_tool0"/>
   <xacro:simple_gripper prefix="right_" parent="right_tool0"/>
 </robot>

Commit message: base plate position off

File: src/ur5_dual_robot_description/urdf/dual_ur5.urdf.xacro (robot description, xacro)
@@ -27,8 +27,8 @@
   <!--
     Arm attachment points: (±0.22, 0, 1.00) world = (±0.22, 0, 0.45) in torso frame.
-    V-shape mount (viewed from behind, i.e. looking along +Y):
-      Left  arm rpy="${pi} ${-pi/4} 0"  → base Z = [+1/√2, 0, -1/√2]  hangs right+down  (\)
-      Right arm rpy="${pi} ${pi/4}  0"  → base Z = [-1/√2, 0, -1/√2]  hangs left+down   (/)
-    The two arms cross inward forming a V.
+    Inverted-V mount (viewed from behind, i.e. looking along +Y):
+      Left  arm at +0.22 rpy="${pi} ${-3*pi/4} 0"  → base Z = [+1/√2, 0, +1/√2]  (\, right+up)
+      Right arm at -0.22 rpy="${pi} ${3*pi/4}  0"  → base Z = [-1/√2, 0, +1/√2]  (/, left+up)
+    Arms splay outward+upward forming Λ from behind.
   -->
   <link name="torso">
@@ -80,5 +80,5 @@
     visual_parameters_file="$(find ur_description)/config/ur5/visual_parameters.yaml"
     generate_ros2_control_tag="false">
-    <origin xyz="-0.22 0 0.45" rpy="${pi} ${-pi/4} 0"/>
+    <origin xyz="0.22 0 0.45" rpy="${pi} ${-3*pi/4} 0"/>
   </xacro:ur_robot>
   <!-- ==================== RIGHT ARM ==================== -->
@@ -93,5 +93,5 @@
     visual_parameters_file="$(find ur_description)/config/ur5/visual_parameters.yaml"
     generate_ros2_control_tag="false">
-    <origin xyz="0.22 0 0.45" rpy="${pi} ${pi/4} 0"/>
+    <origin xyz="-0.22 0 0.45" rpy="${pi} ${3*pi/4} 0"/>
   </xacro:ur_robot>
   <!-- ==================== GRIPPER MACRO ==================== -->

Commit message: robotiq gripper added

File: src/ur5_dual_robot_description/urdf/dual_ur5.urdf.xacro (robot description, xacro)
@@ -48,81 +48,20 @@
   </xacro:ur_robot>
   <!-- ==================== GRIPPER MACRO ==================== -->
-  <xacro:macro name="simple_gripper" params="prefix parent">
-    <link name="${prefix}gripper_base">
-      <visual>
-        <origin xyz="0 0 0.02" rpy="0 0 0"/>
-        <geometry><cylinder radius="0.035" length="0.04"/></geometry>
-        <material name="dark_grey"><color rgba="0.2 0.2 0.2 1"/></material>
-      </visual>
-      <collision>
-        <origin xyz="0 0 0.02" rpy="0 0 0"/>
-        <geometry><cylinder radius="0.035" length="0.04"/></geometry>
-      </collision>
-      <inertial>
-        <mass value="0.3"/>
-        <inertia ixx="0.001" ixy="0" ixz="0" iyy="0.001" iyz="0" izz="0.001"/>
-      </inertial>
-    </link>
-    <joint name="${prefix}gripper_joint" type="fixed">
-      <parent link="${parent}"/>
-      <child link="${prefix}gripper_base"/>
-      <origin xyz="0 0 0" rpy="0 0 0"/>
-    </joint>
-    <link name="${prefix}finger_left">
-      <visual>
-        <origin xyz="0 0 0.02" rpy="0 0 0"/>
-        <geometry><box size="0.012 0.018 0.06"/></geometry>
-        <material name="dark_grey"><color rgba="0.2 0.2 0.2 1"/></material>
-      </visual>
-      <collision>
-        <origin xyz="0 0 0.02" rpy="0 0 0"/>
-        <geometry><box size="0.012 0.018 0.06"/></geometry>
-      </collision>
-      <inertial>
-        <mass value="0.05"/>
-        <inertia ixx="0.0001" ixy="0" ixz="0" iyy="0.0001" iyz="0" izz="0.0001"/>
-      </inertial>
-    </link>
-    <joint name="${prefix}finger_left_joint" type="prismatic">
-      <parent link="${prefix}gripper_base"/>
-      <child link="${prefix}finger_left"/>
-      <origin xyz="-0.025 0 0.04" rpy="0 0 0"/>
-      <axis xyz="1 0 0"/>
-      <limit lower="-0.025" upper="0.0" effort="50" velocity="0.1"/>
-      <dynamics damping="0.1" friction="0.1"/>
-    </joint>
-    <link name="${prefix}finger_right">
-      <visual>
-        <origin xyz="0 0 0.02" rpy="0 0 0"/>
-        <geometry><box size="0.012 0.018 0.06"/></geometry>
-        <material name="dark_grey"><color rgba="0.2 0.2 0.2 1"/></material>
-      </visual>
-      <collision>
-        <origin xyz="0 0 0.02" rpy="0 0 0"/>
-        <geometry><box size="0.012 0.018 0.06"/></geometry>
-      </collision>
-      <inertial>
-        <mass value="0.05"/>
-        <inertia ixx="0.0001" ixy="0" ixz="0" iyy="0.0001" iyz="0" izz="0.0001"/>
-      </inertial>
-    </link>
-    <joint name="${prefix}finger_right_joint" type="prismatic">
-      <parent link="${prefix}gripper_base"/>
-      <child link="${prefix}finger_right"/>
-      <origin xyz="0.025 0 0.04" rpy="0 0 0"/>
-      <axis xyz="1 0 0"/>
-      <limit lower="0.0" upper="0.025" effort="50" velocity="0.1"/>
-      <dynamics damping="0.1" friction="0.1"/>
-    </joint>
-    <!-- TCP (Tool Center Point) — planning target for IK -->
-    <link name="${prefix}tcp"/>
-    <joint name="${prefix}tcp_joint" type="fixed">
-      <parent link="${prefix}gripper_base"/>
-      <child link="${prefix}tcp"/>
-      <origin xyz="0 0 0.1" rpy="0 0 0"/>
-    </joint>
-  </xacro:macro>
-  <!-- ==================== ATTACH GRIPPERS ==================== -->
-  <xacro:simple_gripper prefix="left_" parent="left_tool0"/>
-  <xacro:simple_gripper prefix="right_" parent="right_tool0"/>
+  <xacro:include filename="$(find robotiq_description)/urdf/robotiq_2f_85_macro.urdf.xacro"/>
+  <xacro:include filename="$(find robotiq_description)/urdf/2f_85.ros2_control.xacro"/>
+  <!-- ==================== ROBOTIQ GRIPPERS ==================== -->
+  <xacro:robotiq_gripper
+    name="left_robotiq_2f_85"
+    prefix="left_"
+    parent="left_tool0"
+    include_ros2_control="false">
+    <origin xyz="0 0 0" rpy="0 0 0"/>
+  </xacro:robotiq_gripper>
+  <xacro:robotiq_gripper
+    name="right_robotiq_2f_85"
+    prefix="right_"
+    parent="right_tool0"
+    include_ros2_control="false">
+    <origin xyz="0 0 0" rpy="0 0 0"/>
+  </xacro:robotiq_gripper>
 </robot>

File: src/ur5_dual_robot_moveit_config/config/dual_ur5.ros2_control.xacro (robot description, xacro)
@@ -92,5 +92,6 @@
                 <state_interface name="velocity"/>
             </joint>
-            <joint name="left_finger_left_joint">
+            <!-- Mock Robotiq gripper joints -->
+            <joint name="left_robotiq_85_left_knuckle_joint">
                 <command_interface name="position"/>
                 <state_interface name="position">
@@ -99,19 +100,5 @@
                 <state_interface name="velocity"/>
             </joint>
-            <joint name="left_finger_right_joint">
-                <command_interface name="position"/>
-                <state_interface name="position">
-                  <param name="initial_value">0.0</param>
-                </state_interface>
-                <state_interface name="velocity"/>
-            </joint>
-            <joint name="right_finger_left_joint">
-                <command_interface name="position"/>
-                <state_interface name="position">
-                  <param name="initial_value">0.0</param>
-                </state_interface>
-                <state_interface name="velocity"/>
-            </joint>
-            <joint name="right_finger_right_joint">
+            <joint name="right_robotiq_85_left_knuckle_joint">
                 <command_interface name="position"/>
                 <state_interface name="position">
